Commit message: gps_description:  add urdf generation script

File: romea_gps_description/urdf/gps.xacro (robot description, xacro)
@@ -1,8 +1,7 @@
 <?xml version="1.0"?>
 <robot name="gps" xmlns:xacro="http://www.ros.org/wiki/xacro" >
-  <xacro:macro name="gps_sensor" params="xyz parent_link rate name">
+  <xacro:macro name="gps_sensor" params="xyz parent_link rate name prefix">
     <xacro:property name="link_name" value="${prefix}${name}_link"/>
     <xacro:property name="joint_name" value="${prefix}${name}_joint"/>
-    <xacro:property name="controller_name" value="${prefix}${name}_controller"/>
     <xacro:property name="base_footprint_name" value="${prefix}base_footprint"/>
     <xacro:property name="parent_link_name" value="${prefix}${parent_link}"/>
@@ -75,14 +74,8 @@
           </velocity_sensing>
         </gps>
-       <plugin name="${controller_name}" filename="libgazebo_ros_romea_gps.so">
-         <update_rate>${rate}</update_rate>
-         <body_name>${parent_link}</body_name>
-         <link_name>${link_name}</link_name>
-         <nmea_topic_name>${nmea_topic_name}</nmea_topic_name>
-         <fix_topic_name>${fix_topic_name}</fix_topic_name>
-         <velocity_topic_name>${vel_topic_name}</velocity_topic_name>
-<!--         <antenna_body_position>${xyz}</antenna_body_position>-->
-<!--         <wgs84_anchor>${wgs84_anchor}</wgs84_anchor>-->
-         <gps_name>${prefix}${name}</gps_name>
+       <plugin name="${name}" filename="libromea_gazebo_ros_gps_sensor.so">
+         <ros>
+             <namespace>${prefix}${name}</namespace>
+         </ros>
        </plugin>
       </sensor>

Commit message: update to take into account additional namespace in description

File: romea_gps_description/urdf/gps.xacro (robot description, xacro)
@@ -1,12 +1,13 @@
 <?xml version="1.0"?>
-<robot name="gps" xmlns:xacro="http://www.ros.org/wiki/xacro" >
-  <xacro:macro name="gps_sensor" params="xyz parent_link rate name prefix">
-    <xacro:property name="link_name" value="${prefix}${name}_link"/>
-    <xacro:property name="joint_name" value="${prefix}${name}_joint"/>
-    <xacro:property name="base_footprint_name" value="${prefix}base_footprint"/>
-    <xacro:property name="parent_link_name" value="${prefix}${parent_link}"/>
-    <xacro:property name="nmea_topic_name" value="${name}/nmea_sentence"/>
-    <xacro:property name="fix_topic_name" value="${name}/fix"/>
-    <xacro:property name="vel_topic_name" value="${name}/vel"/>
+<robot name="gps" xmlns:xacro="http://www.ros.org/wiki/xacro">
+  <xacro:macro
+    name="gps_sensor"
+    params="xyz parent_link rate name prefix ros_namespace">
+    <xacro:property name="link_name" value="${prefix}${name}_link" />
+    <xacro:property name="joint_name" value="${prefix}${name}_joint" />
+    <xacro:property name="parent_link_name" value="${prefix}${parent_link}" />
+    <xacro:property name="nmea_topic_name" value="${name}/nmea_sentence" />
+    <xacro:property name="fix_topic_name" value="${name}/fix" />
+    <xacro:property name="vel_topic_name" value="${name}/vel" />
     <gazebo reference="${link_name}">
       <material>Gazebo/White</material>
@@ -14,7 +15,7 @@
     <link name="${link_name}">
       <inertial>
-          <mass value="1" />
-          <origin xyz="0 0 0" rpy="0 0 0" />
-          <inertia ixx="0.000001" ixy="0" ixz="0" iyy="0.000001" iyz="0" izz="0.000001" />
+        <mass value="1" />
+        <origin xyz="0 0 0" rpy="0 0 0" />
+        <inertia ixx="0.000001" ixy="0" ixz="0" iyy="0.000001" iyz="0" izz="0.000001" />
       </inertial>
       <visual>
@@ -74,9 +75,9 @@
           </velocity_sensing>
         </gps>
-       <plugin name="${name}" filename="libromea_gazebo_ros_gps_sensor.so">
-         <ros>
-             <namespace>${prefix}${name}</namespace>
-         </ros>
-       </plugin>
+        <plugin name="driver" filename="libromea_gazebo_ros_gps_sensor.so">
+          <ros>
+            <namespace>${ros_namespace}</namespace>
+          </ros>
+        </plugin>
       </sensor>
     </gazebo>

Commit message: take into account mode into urdf description
Signed-off-by: jean.laneurit <jean.laneurit@inrae.fr>

File: romea_gps_description/urdf/gps.xacro (robot description, xacro)
@@ -3,5 +3,5 @@
   <xacro:macro
     name="gps_sensor"
-    params="xyz parent_link rate name prefix ros_namespace">
+    params="prefix mode xyz parent_link rate name ros_namespace">
     <xacro:property name="link_name" value="${prefix}${name}_link" />
     <xacro:property name="joint_name" value="${prefix}${name}_joint" />
@@ -10,7 +10,7 @@
     <xacro:property name="fix_topic_name" value="${name}/fix" />
     <xacro:property name="vel_topic_name" value="${name}/vel" />
-    <gazebo reference="${link_name}">
-      <material>Gazebo/White</material>
-    </gazebo>
+    <!-- <gazebo reference="${link_name}"> -->
+    <!-- <material>Gazebo/White</material> -->
+    <!-- </gazebo> -->
     <link name="${link_name}">
       <inertial>
@@ -31,55 +31,58 @@
       <child link="${link_name}" />
     </joint>
-    <gazebo reference="${link_name}">
-      <sensor type="gps" name="gps_sensor">
-        <pose>0 0 0 0 0 0</pose>
-        <visualize>0</visualize>
-        <always_on>1</always_on>
-        <update_rate>${rate}</update_rate>
-        <gps>
-          <position_sensing>
-            <horizontal>
-              <noise type="gaussian">
-                <mean>0.0</mean>
-                <stddev>0.0</stddev>
-                <bias_mean>0.0</bias_mean>
-                <bias_stddev>0.0</bias_stddev>
-              </noise>
-            </horizontal>
-            <vertical>
-              <noise type="gaussian">
-                <mean>0.0</mean>
-                <stddev>0.0</stddev>
-                <bias_mean>0.0</bias_mean>
-                <bias_stddev>0.0</bias_stddev>
-              </noise>
-            </vertical>
-          </position_sensing>
-          <velocity_sensing>
-            <horizontal>
-              <noise type="gaussian">
-                <mean>0.0</mean>
-                <stddev>0.0</stddev>
-                <bias_mean>0.0</bias_mean>
-                <bias_stddev>0.0</bias_stddev>
-              </noise>
-            </horizontal>
-            <vertical>
-              <noise type="gaussian">
-                <mean>0.0</mean>
-                <stddev>0.0</stddev>
-                <bias_mean>0.0</bias_mean>
-                <bias_stddev>0.0</bias_stddev>
-              </noise>
-            </vertical>
-          </velocity_sensing>
-        </gps>
-        <plugin name="driver" filename="libromea_gazebo_ros_gps_sensor.so">
-          <ros>
-            <namespace>${ros_namespace}</namespace>
-          </ros>
-        </plugin>
-      </sensor>
-    </gazebo>
+    <xacro:if value="${'simulation' in  mode}">
+      <gazebo reference="${link_name}">
+        <material>Gazebo/White</material>
+        <sensor type="gps" name="gps_sensor">
+          <pose>0 0 0 0 0 0</pose>
+          <visualize>0</visualize>
+          <always_on>1</always_on>
+          <update_rate>${rate}</update_rate>
+          <gps>
+            <position_sensing>
+              <horizontal>
+                <noise type="gaussian">
+                  <mean>0.0</mean>
+                  <stddev>0.0</stddev>
+                  <bias_mean>0.0</bias_mean>
+                  <bias_stddev>0.0</bias_stddev>
+                </noise>
+              </horizontal>
+              <vertical>
+                <noise type="gaussian">
+                  <mean>0.0</mean>
+                  <stddev>0.0</stddev>
+                  <bias_mean>0.0</bias_mean>
+                  <bias_stddev>0.0</bias_stddev>
+                </noise>
+              </vertical>
+            </position_sensing>
+            <velocity_sensing>
+              <horizontal>
+                <noise type="gaussian">
+                  <mean>0.0</mean>
+                  <stddev>0.0</stddev>
+                  <bias_mean>0.0</bias_mean>
+                  <bias_stddev>0.0</bias_stddev>
+                </noise>
+              </horizontal>
+              <vertical>
+                <noise type="gaussian">
+                  <mean>0.0</mean>
+                  <stddev>0.0</stddev>
+                  <bias_mean>0.0</bias_mean>
+                  <bias_stddev>0.0</bias_stddev>
+                </noise>
+              </vertical>
+            </velocity_sensing>
+          </gps>
+          <plugin name="driver" filename="libromea_gazebo_ros_gps_sensor.so">
+            <ros>
+              <namespace>${ros_namespace}</namespace>
+            </ros>
+          </plugin>
+        </sensor>
+      </gazebo>
+    </xacro:if>
   </xacro:macro>
 </robot>

Commit message: description: set Green color to antenna bounding box
Signed-off-by: Jean Laneurit <jean.laneurit@inrae.fr>

File: romea_gps_description/urdf/gps.xacro (robot description, xacro)
@@ -33,5 +33,5 @@
     <xacro:if value="${'simulation' in  mode}">
       <gazebo reference="${link_name}">
-        <material>Gazebo/White</material>
+        <material>Gazebo/Green</material>
         <sensor type="gps" name="gps_sensor">
           <pose>0 0 0 0 0 0</pose>

Commit message: description: add gps_simulation xacro file
Signed-off-by: Jean Laneurit <jean.laneurit@inrae.fr>

File: romea_gps_description/urdf/gps.xacro (robot description, xacro)
@@ -32,58 +32,13 @@
     </joint>
     <xacro:if value="${'simulation' in  mode}">
-      <gazebo reference="${link_name}">
-        <material>Gazebo/Green</material>
-        <sensor type="gps" name="gps_sensor">
-          <pose>0 0 0 0 0 0</pose>
-          <visualize>0</visualize>
-          <always_on>1</always_on>
-          <update_rate>${rate}</update_rate>
-          <gps>
-            <position_sensing>
-              <horizontal>
-                <noise type="gaussian">
-                  <mean>0.0</mean>
-                  <stddev>0.0</stddev>
-                  <bias_mean>0.0</bias_mean>
-                  <bias_stddev>0.0</bias_stddev>
-                </noise>
-              </horizontal>
-              <vertical>
-                <noise type="gaussian">
-                  <mean>0.0</mean>
-                  <stddev>0.0</stddev>
-                  <bias_mean>0.0</bias_mean>
-                  <bias_stddev>0.0</bias_stddev>
-                </noise>
-              </vertical>
-            </position_sensing>
-            <velocity_sensing>
-              <horizontal>
-                <noise type="gaussian">
-                  <mean>0.0</mean>
-                  <stddev>0.0</stddev>
-                  <bias_mean>0.0</bias_mean>
-                  <bias_stddev>0.0</bias_stddev>
-                </noise>
-              </horizontal>
-              <vertical>
-                <noise type="gaussian">
-                  <mean>0.0</mean>
-                  <stddev>0.0</stddev>
-                  <bias_mean>0.0</bias_mean>
-                  <bias_stddev>0.0</bias_stddev>
-                </noise>
-              </vertical>
-            </velocity_sensing>
-          </gps>
-          <plugin name="driver" filename="libromea_gazebo_ros_gps_sensor.so">
-            <ros>
-              <namespace>${ros_namespace}</namespace>
-            </ros>
-            <frame_name>${link_name}</frame_name>
-            <dual_antenna>${dual_antenna}</dual_antenna>
-          </plugin>
-        </sensor>
-      </gazebo>
+      <xacro:include filename="$(find romea_gps_description)/urdf/gps.simulation.xacro" />
+      <xacro:gps_sensor_simulation
+        prefix="${prefix}"
+        mode="${mode}"
+        name="${name}"
+        rate="${rate}"
+        link_name="${link_name}"
+        dual_antenna="${dual_antenna}"
+        ros_namespace="${ros_namespace}"/>
     </xacro:if>
   </xacro:macro>
