Commit message: add antenna geometry description
Signed-off-by: jean.laneurit <jean.laneurit@inrae.fr>

File: romea_gps_description/urdf/gps.simulation.xacro (robot description, xacro)
@@ -3,5 +3,9 @@
   <xacro:macro
     name="gps_sensor_simulation"
-    params="prefix mode link_name rate name dual_antenna ros_namespace">
+    params="prefix mode link_name name configuration ros_namespace">
+    <xacro:property name="rate"
+      value="${configuration['rate']}" />
+    <xacro:property name="dual_antenna"
+      value="${configuration['dual_antenna']}" />
     <xacro:if value="${'gazebo' in  mode}">
       <gazebo reference="${link_name}">

File: romea_gps_description/urdf/gps.xacro (robot description, xacro)
@@ -1,31 +1,84 @@
 <?xml version="1.0"?>
 <robot name="gps" xmlns:xacro="http://www.ros.org/wiki/xacro">
-  <xacro:macro
-    name="gps_sensor"
-    params="prefix mode xyz parent_link rate dual_antenna name ros_namespace">
-    <xacro:property name="link_name" value="${prefix}${name}_link" />
-    <xacro:property name="joint_name" value="${prefix}${name}_joint" />
-    <xacro:property name="parent_link_name" value="${prefix}${parent_link}" />
-    <xacro:property name="nmea_topic_name" value="${name}/nmea_sentence" />
-    <xacro:property name="fix_topic_name" value="${name}/fix" />
-    <xacro:property name="vel_topic_name" value="${name}/vel" />
-    <!-- <gazebo reference="${link_name}"> -->
-    <!-- <material>Gazebo/White</material> -->
-    <!-- </gazebo> -->
+  <xacro:macro name="gps_sensor"
+    params="prefix mode name configuration geometry mesh_visual ros_namespace">
+    <xacro:property name="link_name"
+      value="${prefix}${name}_link" />
+    <xacro:property name="joint_name"
+      value="${prefix}${name}_joint" />
+    <xacro:property name="parent_link_name"
+      value="${prefix}${configuration['parent_link']}" />
+    <xacro:property name="xyz"
+      value="${configuration['xyz']}" />
+    <xacro:property name="mass"
+      value="${geometry['mass']}" />
+    <xacro:property name="shape"
+      value="${geometry['shape']}" />
+    <xacro:property name="aabb_length"
+      value="${geometry['aabb']['length']}" />
+    <xacro:property name="aabb_width"
+      value="${geometry['aabb']['width']}" />
+    <xacro:property name="aabb_height"
+      value="${geometry['aabb']['height']}" />
+    <xacro:property name="aabb_center"
+      value="${geometry['aabb']['center']}" />
+    <xacro:if value="${mesh_visual == True and 'mesh' in geometry}">
+      <xacro:property name="mesh_xyz"
+        value="${geometry['mesh']['xyz']}" />
+      <xacro:property name="mesh_rpy"
+        value="${geometry['mesh']['rpy']}" />
+      <xacro:property name="mesh_scale"
+        value="${geometry['mesh']['scale']}" />
+      <xacro:property name="mesh_filename"
+        value="${geometry['mesh']['filename']}" />
+    </xacro:if>
+    <xacro:property name="nmea_topic_name"
+      value="${name}/nmea_sentence" />
+    <xacro:property name="fix_topic_name"
+      value="${name}/fix" />
+    <xacro:property name="vel_topic_name"
+      value="${name}/vel" />
     <link name="${link_name}">
       <inertial>
-        <mass value="1" />
-        <origin xyz="0 0 0" rpy="0 0 0" />
-        <inertia ixx="0.000001" ixy="0" ixz="0" iyy="0.000001" iyz="0" izz="0.000001" />
+        <mass value="${mass}" />
+        <origin xyz="${aabb_center[0]} ${aabb_center[1]} ${aabb_center[2]}" />
+        <inertia ixx="${0.0833333 * mass * (aabb_width*aabb_width + aabb_height*aabb_height)}"
+          ixy="0.0" ixz="0.0"
+          iyy="${0.0833333 * mass * (aabb_height*aabb_height + aabb_length*aabb_length)}" iyz="0.0"
+          izz="${0.0833333 * mass * (aabb_length*aabb_length + aabb_width*aabb_width)}" />
       </inertial>
       <visual>
-        <origin xyz="0 0 0" rpy="0 0 0" />
+        <xacro:if value="${mesh_visual == True and 'mesh' in geometry}">
+          <origin xyz="${mesh_xyz[0]} ${mesh_xyz[1]} ${mesh_xyz[2]}"
+            rpy="${mesh_rpy[0]/180.*pi} ${mesh_rpy[1]/180.*pi} ${mesh_rpy[2]/180.*pi}" />
+          <geometry>
+            <mesh filename="${mesh_filename}"
+              scale="${mesh_scale[0]} ${mesh_scale[1]} ${mesh_scale[2]}" />
+          </geometry>
+        </xacro:if>
+        <xacro:if value="${mesh_visual == False or 'mesh' not in geometry}">
+          <origin xyz="${aabb_center[0]} ${aabb_center[1]} ${aabb_center[2]}" rpy="0 0 0" />
+          <xacro:if value="${shape == 'disk'}">
+            <geometry>
+              <cylinder length="${aabb_height}" radius="${aabb_length / 2.0}" />
+            </geometry>
+          </xacro:if>
+          <xacro:if value="${shape == 'patch'}">
+            <geometry>
+              <box size="${aabb_length} ${aabb_width} ${aabb_height}" />
+            </geometry>
+          </xacro:if>
+        </xacro:if>
+      </visual>
+      <!-- <collision>
+        <origin xyz="${aabb_center[0]} ${aabb_center[1]} ${aabb_center[2]}" rpy="0 0 0" />
         <geometry>
-          <cylinder length="0.05" radius="0.1" />
+          <box size="${aabb_length} ${aabb_width} ${aabb_height}" />
         </geometry>
-      </visual>
+      </collision> -->
     </link>
-    <joint name="${joint_name}" type="fixed">
-      <origin xyz="${xyz}" rpy="0 0 0" />
+    <joint
+      name="${joint_name}" type="fixed">
+      <origin xyz="${xyz[0]} ${xyz[1]} ${xyz[2]}" rpy="0 0 0" />
       <parent link="${parent_link_name}" />
       <child link="${link_name}" />
@@ -37,8 +90,7 @@
         mode="${mode}"
         name="${name}"
-        rate="${rate}"
         link_name="${link_name}"
-        dual_antenna="${dual_antenna}"
-        ros_namespace="${ros_namespace}"/>
+        configuration="${configuration}"
+        ros_namespace="${ros_namespace}" />
     </xacro:if>
   </xacro:macro>

Commit message: refactoring
Signed-off-by: Jean Laneurit <jean.laneurit@inrae.fr>

File: romea_gps_description/urdf/gps.simulation.xacro (robot description, xacro)
@@ -1,4 +1,43 @@
 <?xml version="1.0"?>
+<!-- <sensor name="custom_odometer" type="custom" gz:type="odometer"> -->
 <robot name="gps" xmlns:xacro="http://www.ros.org/wiki/xacro">
+  <xacro:macro name="common_sensing">
+    <position_sensing>
+      <horizontal>
+        <noise type="gaussian">
+          <mean>0.1</mean>
+          <stddev>0.0</stddev>
+          <bias_mean>0.0</bias_mean>
+          <bias_stddev>0.0</bias_stddev>
+        </noise>
+      </horizontal>
+      <vertical>
+        <noise type="gaussian">
+          <mean>0.1</mean>
+          <stddev>0.0</stddev>
+          <bias_mean>0.0</bias_mean>
+          <bias_stddev>0.0</bias_stddev>
+        </noise>
+      </vertical>
+    </position_sensing>
+    <velocity_sensing>
+      <horizontal>
+        <noise type="gaussian">
+          <mean>0.1</mean>
+          <stddev>0.0</stddev>
+          <bias_mean>0.0</bias_mean>
+          <bias_stddev>0.0</bias_stddev>
+        </noise>
+      </horizontal>
+      <vertical>
+        <noise type="gaussian">
+          <mean>0.1</mean>
+          <stddev>0.0</stddev>
+          <bias_mean>0.0</bias_mean>
+          <bias_stddev>0.0</bias_stddev>
+        </noise>
+      </vertical>
+    </velocity_sensing>
+  </xacro:macro>
   <xacro:macro
     name="gps_sensor_simulation"
@@ -8,53 +47,23 @@
     <xacro:property name="dual_antenna"
       value="${configuration['dual_antenna']}" />
+    <!-- <xacro:if value="${'classic' in mode}">
+      <xacro:property name="sensor_type" value="gps" />
+    </xacro:if>
+    <xacro:if
+      value="${'classic' not in mode}">
+      <xacro:property name="sensor_type" value="custom" />
+    </xacro:if> -->
     <xacro:if value="${'gazebo' in  mode}">
       <gazebo reference="${link_name}">
         <material>Gazebo/Green</material>
-        <sensor type="gps" name="gps_sensor">
+        <sensor type="custom" name="gps_sensor" gz:type="gps"
+          xmlns:gz="http://gazebosim.org/schema/gz">
           <pose>0 0 0 0 0 0</pose>
           <always_on>1</always_on>
           <update_rate>${rate}</update_rate>
-          <topic>${ros_namespace}/navsat</topic>
-          <gz_frame_id>${link_name}</gz_frame_id>  <!-- used only with gazebo 6 or lower -->
-          <ignition_frame_id>${link_name}</ignition_frame_id> <!-- used by gazebo 7 or higher-->
-          <gps>
-            <position_sensing>
-              <horizontal>
-                <noise type="gaussian">
-                  <mean>0.0</mean>
-                  <stddev>0.0</stddev>
-                  <bias_mean>0.0</bias_mean>
-                  <bias_stddev>0.0</bias_stddev>
-                </noise>
-              </horizontal>
-              <vertical>
-                <noise type="gaussian">
-                  <mean>0.0</mean>
-                  <stddev>0.0</stddev>
-                  <bias_mean>0.0</bias_mean>
-                  <bias_stddev>0.0</bias_stddev>
-                </noise>
-              </vertical>
-            </position_sensing>
-            <velocity_sensing>
-              <horizontal>
-                <noise type="gaussian">
-                  <mean>0.0</mean>
-                  <stddev>0.0</stddev>
-                  <bias_mean>0.0</bias_mean>
-                  <bias_stddev>0.0</bias_stddev>
-                </noise>
-              </horizontal>
-              <vertical>
-                <noise type="gaussian">
-                  <mean>0.0</mean>
-                  <stddev>0.0</stddev>
-                  <bias_mean>0.0</bias_mean>
-                  <bias_stddev>0.0</bias_stddev>
-                </noise>
-              </vertical>
-            </velocity_sensing>
-          </gps>
-          <xacro:if value="${'classic' in mode}">
+          <!-- <xacro:if value="${'classic' in mode}">
+            <gps>
+              <xacro:common_sensing />
+            </gps>
             <plugin name="driver" filename="libromea_gazebo_ros_gps_sensor.so">
               <ros>
@@ -64,5 +73,14 @@
               <dual_antenna>${dual_antenna}</dual_antenna>
             </plugin>
-          </xacro:if>
+          </xacro:if> -->
+          <!-- <xacro:if value="${'classic' not in mode}"> -->
+          <topic>${ros_namespace}/nmea</topic>
+          <gz_frame_id>${link_name}</gz_frame_id>
+          <ignition_frame_id>${link_name}</ignition_frame_id>
+          <gz:gps>
+            <xacro:common_sensing />
+          </gz:gps>
+          <plugin filename="romea_gps_gazebo" name="romea::gz::NmeaGps" />
+          <!-- </xacro:if> -->
         </sensor>
       </gazebo>

Commit message: fix linter errors
Signed-off-by: Jean Laneurit <jean.laneurit@inrae.fr>

File: romea_gps_description/urdf/gps.simulation.xacro (robot description, xacro)
@@ -47,20 +47,12 @@
     <xacro:property name="dual_antenna"
       value="${configuration['dual_antenna']}" />
-    <!-- <xacro:if value="${'classic' in mode}">
-      <xacro:property name="sensor_type" value="gps" />
-    </xacro:if>
-    <xacro:if
-      value="${'classic' not in mode}">
-      <xacro:property name="sensor_type" value="custom" />
-    </xacro:if> -->
     <xacro:if value="${'gazebo' in  mode}">
       <gazebo reference="${link_name}">
         <material>Gazebo/Green</material>
-        <sensor type="custom" name="gps_sensor" gz:type="gps"
-          xmlns:gz="http://gazebosim.org/schema/gz">
-          <pose>0 0 0 0 0 0</pose>
-          <always_on>1</always_on>
-          <update_rate>${rate}</update_rate>
-          <!-- <xacro:if value="${'classic' in mode}">
+        <xacro:if value="${'classic' in mode}">
+          <sensor type="gps" name="gps_sensor">
+            <pose>0 0 0 0 0 0</pose>
+            <always_on>1</always_on>
+            <update_rate>${rate}</update_rate>
             <gps>
               <xacro:common_sensing />
@@ -73,15 +65,22 @@
               <dual_antenna>${dual_antenna}</dual_antenna>
             </plugin>
-          </xacro:if> -->
-          <!-- <xacro:if value="${'classic' not in mode}"> -->
-          <topic>${ros_namespace}/nmea</topic>
-          <gz_frame_id>${link_name}</gz_frame_id>
-          <ignition_frame_id>${link_name}</ignition_frame_id>
-          <gz:gps>
-            <xacro:common_sensing />
-          </gz:gps>
-          <plugin filename="romea_gps_gazebo" name="romea::gz::NmeaGps" />
-          <!-- </xacro:if> -->
-        </sensor>
+          </sensor>
+        </xacro:if>
+        <xacro:if value="${'classic' not in mode}">
+          <sensor type="custom" name="gps_sensor" gz:type="gps"
+            xmlns:gz="http://gazebosim.org/schema/gz">
+            <pose>0 0 0 0 0 0</pose>
+            <always_on>1</always_on>
+            <update_rate>${rate}</update_rate>
+            <topic>${ros_namespace}/nmea</topic>
+            <gz_frame_id>${link_name}</gz_frame_id>
+            <ignition_frame_id>${link_name}</ignition_frame_id>
+            <dual_antenna>${dual_antenna}</dual_antenna>
+            <gz:gps>
+              <xacro:common_sensing />
+            </gz:gps>
+            <plugin filename="romea_gps_gazebo" name="romea::gz::NmeaGps" />
+          </sensor>
+        </xacro:if>
       </gazebo>
     </xacro:if>

Commit message: gps_description: add standalone option xacro files
Signed-off-by: Jean Laneurit <jean.laneurit@inrae.fr>

File: romea_gps_description/urdf/gps.simulation.xacro (robot description, xacro)
@@ -80,5 +80,5 @@
               <xacro:common_sensing />
             </gz:gps>
-            <plugin filename="romea_gps_gazebo" name="romea::gz::NmeaGps" />
+            <plugin filename="romea_gps_gazebo_plugin" name="romea::gz::NmeaGps" />
           </sensor>
         </xacro:if>

File: romea_gps_description/urdf/gps.xacro (robot description, xacro)
@@ -2,5 +2,5 @@
 <robot name="gps" xmlns:xacro="http://www.ros.org/wiki/xacro">
   <xacro:macro name="gps_sensor"
-    params="prefix mode name configuration geometry mesh_visual ros_namespace">
+    params="prefix mode name configuration geometry mesh_visual ros_namespace standalone">
     <xacro:property name="link_name"
       value="${prefix}${name}_link" />
@@ -78,10 +78,12 @@
       </collision> -->
     </link>
-    <joint
-      name="${joint_name}" type="fixed">
-      <origin xyz="${xyz[0]} ${xyz[1]} ${xyz[2]}" rpy="0 0 0" />
-      <parent link="${parent_link_name}" />
-      <child link="${link_name}" />
-    </joint>
+    <xacro:if value="${standalone == False}">
+      <joint
+        name="${joint_name}" type="fixed">
+        <origin xyz="${xyz[0]} ${xyz[1]} ${xyz[2]}" rpy="0 0 0" />
+        <parent link="${parent_link_name}" />
+        <child link="${link_name}" />
+      </joint>
+    </xacro:if>
     <xacro:if value="${'simulation' in  mode}">
       <xacro:include filename="$(find romea_gps_description)/urdf/gps.simulation.xacro" />
